File: electronics/front-end.kicad_sch (KiCad schematic)
At the start: 47 parts, among them K1 HF49FD_005-1H12T, Q1 MMBT2222A, U6 ISO1540, U7 ADS1115IDGS, U8 INA240A2D

Commit message: Add current-sense amplifier offset and fix first-boot download mode
Improve measurement accuracy near zero and enable bidirectional current sensing by adding the current-sense amplifier offset.

Resolve the download-mode issue encountered on first boot.

Signed-off-by: Maxim Pavlov <max.eelabs@gmail.com>
Parts:
- added C24: 100nF, Capacitor_SMD:C_0805_2012Metric, symbol Device:C
- added R27: 22k, Resistor_SMD:R_0805_2012Metric, symbol Device:R
- added R28: 2k, Resistor_SMD:R_0805_2012Metric, symbol Device:R
- added U10: LM321, Package_TO_SOT_SMD:SOT-23-5, symbol Amplifier_Operational:LM321
- renumbered C24 to C25, C25 to C26, C26 to C27, C27 to C28, C28 to C29, C29 to C30, C30 to C31, R27 to R29, R28 to R30, R29 to R31, R30 to R32, R31 to R33, R32 to R34, R33 to R35, R34 to R36, R35 to R37, R36 to R38, R37 to R39, R38 to R40, R39 to R41, R40 to R42, R41 to R43, R42 to R44
Connections:
- net GNDS: now also C24.2, R28.2, U10.2 (V-); no longer U8.7 (REF1)
- net V3.3-F: now also C24.1, R27.1, U10.5 (V+)
- new net: R27.2, R28.1, U10.1 (+)
- new net: U10.3 (-), U10.4, U8.7 (REF1)
Other:
- moved on the sheet: C22, C23, C25, R25, R26, R29, TP7, U7
