File: electronics/power.kicad_sch (KiCad schematic)
At the start: 14 parts, among them U3 LD1117S33, U4 LD1117S33

Commit message: Added IO3 pullup and negative 3V3 rail testpoint, few other PCB layput improvements.
Parts:
- C7, C8: value 330p 1kV -> 330p
Changed lines of the file:
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@@
 		(title "PSU-EXT Power")
 		(date "2026-08-08")
-		(rev "1.3.0")
+		(rev "1.3.1")
 		(company "MaxEELabs")
 		(comment 3 "This hardware design is licensed under CERN-OHL-S v2.\nCopyright © 2026 PSU-EXT Authors: https://github.com/PSU-Ext-Org")
@@
 			)
 		)
-		(property "Value" "330p 1kV"
+		(property "Value" "330p"
 			(at 139.7 71.12 90)
 			(show_name no)
@@
 			)
 		)
-		(property "Description" "Unpolarized capacitor"
+		(property "Description" "Unpolarized capacitor  1kV"
 			(at 139.7 76.2 0)
 			(hide yes)
@@
 			)
 		)
-		(property "Value" "330p 1kV"
+		(property "Value" "330p"
 			(at 139.7 33.02 90)
 			(show_name no)
@@
 			)
 		)
-		(property "Description" "Unpolarized capacitor"
+		(property "Description" "Unpolarized capacitor 1kV"
 			(at 139.7 38.1 0)
 			(hide yes)
