File: electronics/front-end-voltage.kicad_sch (KiCad schematic)
At the start: 21 parts, among them U11 TSZ122IYDT, U12 LM2664M6

Commit message: Added IO3 pullup and negative 3V3 rail testpoint, few other PCB layput improvements.
Parts:
- added TP7: -3V3, TestPoint:TestPoint_Pad_D1.5mm, symbol Connector:TestPoint
Connections:
- net -3V3: now also TP7.1
Changed lines of the file:
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@@
 		(title "PSU-EXT Front-End. Volatge ")
 		(date "2026-08-08")
-		(rev "1.3.0")
+		(rev "1.3.1")
 		(company "MaxEELabs")
 		(comment 3 "This hardware design is licensed under CERN-OHL-S v2.\nCopyright © 2026 PSU-EXT Authors: https://github.com/PSU-Ext-Org")
@@
 		(pts
 			(xy 222.25 54.61) (xy 227.33 54.61)
+		)
+		(stroke
+			(width 0)
+			(type default)
+		)
+	)
+	(wire
+		(pts
+			(xy 251.46 38.1) (xy 251.46 39.37)
 		)
 		(stroke
@@
 					(unit 1)
 				)
+			)
+		)
+	)
+	(symbol
+		(lib_id "Connector:TestPoint")
+		(at 251.46 38.1 0)
+		(unit 1)
+		(body_style 1)
+		(exclude_from_sim no)
+		(in_bom yes)
+		(on_board yes)
+		(in_pos_files yes)
+		(dnp no)
+		(fields_autoplaced yes)
+		(property "Reference" "TP7"
+			(at 254 33.5279 0)
+			(show_name no)
+			(do_not_autoplace no)
+			(effects
+				(font
+					(size 1.27 1.27)
+				)
+				(justify left)
+			)
+		)
+		(property "Value" "-3V3"
+			(at 254 36.0679 0)
+			(show_name no)
+			(do_not_autoplace no)
+			(effects
+				(font
+					(size 1.27 1.27)
+				)
+				(justify left)
+			)
+		)
+		(property "Footprint" "TestPoint:TestPoint_Pad_D1.5mm"
+			(at 256.54 38.1 0)
+			(hide yes)
+			(show_name no)
+			(do_not_autoplace no)
+			(effects
+				(font
+					(size 1.27 1.27)
+				)
+			)
+		)
+		(property "Datasheet" ""
+			(at 256.54 38.1 0)
+			(hide yes)
+			(show_name no)
+			(do_not_autoplace no)
+			(effects
+				(font
+					(size 1.27 1.27)
+				)
+			)
+		)
+		(property "Description" "test point"
+			(at 251.46 38.1 0)
+			(hide yes)
+			(show_name no)
+			(do_not_autoplace no)
+			(effects
+				(font
+					(size 1.27 1.27)
+				)
+			)
+		)
+		(pin "1"
+		)
+		(instances
+			(project "psu-ext"
+				(path "/3cca1064-5b2a-48a0-8872-f4d00db38e9c/284031bb-95f3-41d1-9c76-36a65272dfe7"
+					(reference "TP7")
+					(unit 1)
+				)

Commit message: Fixex for proect before PCBA. TODO. BOM, CPL, EXPORT
Parts:
- TP7: now left out of the parts list
- renumbered R36 to R37, R37 to R38, R38 to R39, R39 to R40, R40 to R41, R41 to R42, R42 to R43, R43 to R44, R44 to R45, R45 to R46
Changed lines of the file:
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@@
 		(dnp no)
 		(fields_autoplaced yes)
-		(property "Reference" "R37"
+		(property "Reference" "R38"
 			(at 49.53 27.94 90)
 			(show_name no)
@@
 			(project "psu-ext"
 				(path "/3cca1064-5b2a-48a0-8872-f4d00db38e9c/284031bb-95f3-41d1-9c76-36a65272dfe7"
-					(reference "R37")
+					(reference "R38")
 					(unit 1)
 				)
@@
 		(in_pos_files yes)
 		(dnp no)
-		(property "Reference" "R45"
+		(property "Reference" "R46"
 			(at 123.19 81.28 90)
 			(show_name no)
@@
 			(project "psu-ext"
 				(path "/3cca1064-5b2a-48a0-8872-f4d00db38e9c/284031bb-95f3-41d1-9c76-36a65272dfe7"
-					(reference "R45")
+					(reference "R46")
 					(unit 1)
 				)
@@
 		(dnp no)
 		(fields_autoplaced yes)
-		(property "Reference" "R38"
+		(property "Reference" "R39"
 			(at 58.42 78.74 90)
 			(show_name no)
@@
 			(project "psu-ext"
 				(path "/3cca1064-5b2a-48a0-8872-f4d00db38e9c/284031bb-95f3-41d1-9c76-36a65272dfe7"
-					(reference "R38")
+					(reference "R39")
 					(unit 1)
 				)
@@
 		(body_style 1)
 		(exclude_from_sim no)
-		(in_bom yes)
-		(on_board yes)
-		(in_pos_files yes)
+		(in_bom no)
+		(on_board yes)
+		(in_pos_files no)
 		(dnp no)
 		(fields_autoplaced yes)
@@
 		(dnp no)
 		(fields_autoplaced yes)
-		(property "Reference" "R36"
+		(property "Reference" "R37"
 			(at 48.26 78.74 90)
 			(show_name no)
@@
 			(project "psu-ext"
 				(path "/3cca1064-5b2a-48a0-8872-f4d00db38e9c/284031bb-95f3-41d1-9c76-36a65272dfe7"
-					(reference "R36")
+					(reference "R37")
 					(unit 1)
 				)
@@
 		(dnp no)
 		(fields_autoplaced yes)
-		(property "Reference" "R39"
+		(property "Reference" "R40"
 			(at 59.69 27.94 90)
 			(show_name no)
@@
 			(project "psu-ext"
 				(path "/3cca1064-5b2a-48a0-8872-f4d00db38e9c/284031bb-95f3-41d1-9c76-36a65272dfe7"
-					(reference "R39")
+					(reference "R40")
 					(unit 1)
 				)
@@
 		(in_pos_files yes)
 		(dnp no)
-		(property "Reference" "R40"
+		(property "Reference" "R41"
 			(at 58.674 90.17 0)
 			(show_name no)
@@
 			(project "psu-ext"
 				(path "/3cca1064-5b2a-48a0-8872-f4d00db38e9c/284031bb-95f3-41d1-9c76-36a65272dfe7"
-					(reference "R40")
+					(reference "R41")
 					(unit 1)
 				)
@@
 		(in_pos_files yes)
 		(dnp no)
-		(property "Reference" "R41"
+		(property "Reference" "R42"
 			(at 60.452 39.37 0)
 			(show_name no)
@@
 			(project "psu-ext"
 				(path "/3cca1064-5b2a-48a0-8872-f4d00db38e9c/284031bb-95f3-41d1-9c76-36a65272dfe7"
-					(reference "R41")
+					(reference "R42")
 					(unit 1)
 				)
@@
 		(dnp no)
 		(fields_autoplaced yes)
-		(property "Reference" "R42"
+		(property "Reference" "R43"
 			(at 110.49 54.6099 0)
 			(show_name no)
@@
 			(project "psu-ext"
 				(path "/3cca1064-5b2a-48a0-8872-f4d00db38e9c/284031bb-95f3-41d1-9c76-36a65272dfe7"
-					(reference "R42")
+					(reference "R43")
 					(unit 1)
 				)
@@
 		(in_pos_files yes)
 		(dnp no)
-		(property "Reference" "R44"
+		(property "Reference" "R45"
 			(at 123.19 30.48 90)
 			(show_name no)
@@
 			(project "psu-ext"
 				(path "/3cca1064-5b2a-48a0-8872-f4d00db38e9c/284031bb-95f3-41d1-9c76-36a65272dfe7"
-					(reference "R44")
+					(reference "R45")
 					(unit 1)
 				)
@@
 		(dnp no)
 		(fields_autoplaced yes)
-		(property "Reference" "R43"
+		(property "Reference" "R44"
 			(at 110.49 105.4099 0)
 			(show_name no)
@@
 			(project "psu-ext"
 				(path "/3cca1064-5b2a-48a0-8872-f4d00db38e9c/284031bb-95f3-41d1-9c76-36a65272dfe7"
-					(reference "R43")
-					(unit 1)
-				)
+					(reference "R44")
+					(unit 1)
+				)
