File: electronics/front-end-adc-c.kicad_sch (KiCad schematic)
At the start: 39 parts, among them K1 HF49FD_005-1H12T, Q1 MMBT2222A, U10 INA240A2D, U7 ISO1540, U8 ADS1115IDGS, U9 LM321

Commit message: Added IO3 pullup and negative 3V3 rail testpoint, few other PCB laypu… (#4)
* Added IO3 pullup and negative 3V3 rail testpoint, few other PCB layput improvements.
* Updated exports - gerbers, schematics, bom, CPL KiCad for version 1.3.1

---------

Signed-off-by: Maxim Pavlov <max.eelabs@gmail.com>
Parts:
- C29: now not fitted; now left out of the parts list
- R31: renamed from R30; value 22k -> 20k
- R36: renamed from R35; now not fitted; now left out of the parts list
- renumbered R23 to R24, R24 to R25, R25 to R26, R26 to R27, R27 to R28, R28 to R29, R29 to R30, R31 to R32, R32 to R33, R33 to R34, R34 to R35
Changed lines of the file:
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@@
 		(title "PSU-EXT Front-End. ADC, relay amd current sense")
 		(date "2026-08-08")
-		(rev "1.3.0")
+		(rev "1.3.1")
 		(company "MaxEELabs")
 		(comment 3 "This hardware design is licensed under CERN-OHL-S v2.\nCopyright © 2026 PSU-EXT Authors: https://github.com/PSU-Ext-Org")
@@
 		(in_bom no)
 		(on_board yes)
-		(in_pos_files yes)
+		(in_pos_files no)
 		(dnp no)
 		(property "Reference" "H10"
@@
 		(dnp no)
 		(fields_autoplaced yes)
-		(property "Reference" "R26"
+		(property "Reference" "R27"
 			(at 85.09 38.0999 0)
 			(show_name no)
@@
 			(project "psu-ext"
 				(path "/3cca1064-5b2a-48a0-8872-f4d00db38e9c/8382cf51-befd-44eb-9cec-01756b7c42d3"
-					(reference "R26")
+					(reference "R27")
 					(unit 1)
 				)
@@
 		(body_style 1)
 		(exclude_from_sim no)
-		(in_bom yes)
+		(in_bom no)
 		(on_board yes)
-		(in_pos_files yes)
-		(dnp no)
-		(property "Reference" "R35"
+		(in_pos_files no)
+		(dnp yes)
+		(property "Reference" "R36"
 			(at 261.366 124.46 90)
 			(show_name no)
@@
 			(project "psu-ext"
 				(path "/3cca1064-5b2a-48a0-8872-f4d00db38e9c/8382cf51-befd-44eb-9cec-01756b7c42d3"
-					(reference "R35")
+					(reference "R36")
 					(unit 1)
 				)
@@
 		(in_bom no)
 		(on_board yes)
-		(in_pos_files yes)
+		(in_pos_files no)
 		(dnp no)
 		(property "Reference" "H8"
@@
 		(dnp no)
 		(fields_autoplaced yes)
-		(property "Reference" "R27"
+		(property "Reference" "R28"
 			(at 93.98 38.0999 0)
 			(show_name no)
@@
 			(project "psu-ext"
 				(path "/3cca1064-5b2a-48a0-8872-f4d00db38e9c/8382cf51-befd-44eb-9cec-01756b7c42d3"
-					(reference "R27")
+					(reference "R28")
 					(unit 1)
 				)
@@
 		(dnp no)
 		(fields_autoplaced yes)
-		(property "Reference" "R30"
+		(property "Reference" "R31"
 			(at 180.34 43.1799 0)
 			(show_name no)
@@
 			)
 		)
-		(property "Value" "22k"
+		(property "Value" "20k"
 			(at 180.34 45.7199 0)
 			(show_name no)
@@
 			(project "psu-ext"
 				(path "/3cca1064-5b2a-48a0-8872-f4d00db38e9c/8382cf51-befd-44eb-9cec-01756b7c42d3"
-					(reference "R30")
+					(reference "R31")
 					(unit 1)
 				)
@@
 		(in_pos_files yes)
 		(dnp no)
-		(property "Reference" "R33"
+		(property "Reference" "R34"
 			(at 190.5 140.97 90)
 			(show_name no)
@@
 			(project "psu-ext"
 				(path "/3cca1064-5b2a-48a0-8872-f4d00db38e9c/8382cf51-befd-44eb-9cec-01756b7c42d3"
-					(reference "R33")
+					(reference "R34")
 					(unit 1)
 				)
@@
 		(body_style 1)
 		(exclude_from_sim no)
-		(in_bom yes)
+		(in_bom no)
 		(on_board yes)
-		(in_pos_files yes)
-		(dnp no)
+		(in_pos_files no)
+		(dnp yes)
 		(property "Reference" "C29"
 			(at 261.366 134.62 90)
@@
 		(dnp no)
 		(fields_autoplaced yes)
-		(property "Reference" "R23"
+		(property "Reference" "R24"
 			(at 45.72 109.22 90)
 			(show_name no)
@@
 			(project "psu-ext"
 				(path "/3cca1064-5b2a-48a0-8872-f4d00db38e9c/8382cf51-befd-44eb-9cec-01756b7c42d3"
-					(reference "R23")
+					(reference "R24")
 					(unit 1)
 				)
@@
 		(dnp no)
 		(fields_autoplaced yes)
-		(property "Reference" "R28"
+		(property "Reference" "R29"
 			(at 133.35 34.2899 0)
 			(show_name no)
@@
 			(project "psu-ext"
 				(path "/3cca1064-5b2a-48a0-8872-f4d00db38e9c/8382cf51-befd-44eb-9cec-01756b7c42d3"
-					(reference "R28")
+					(reference "R29")
 					(unit 1)
 				)
@@
 		)
 		(property "Value" "INA240A2D"
-			(at 247.142 40.386 0)
+			(at 246.634 40.386 0)
 			(show_name no)
 			(do_not_autoplace no)
@@
 		(in_pos_files yes)
 		(dnp no)
-		(property "Reference" "R29"
+		(property "Reference" "R30"
 			(at 138.938 109.474 90)
 			(show_name no)
@@
 			(project "psu-ext"
 				(path "/3cca1064-5b2a-48a0-8872-f4d00db38e9c/8382cf51-befd-44eb-9cec-01756b7c42d3"
-					(reference "R29")
+					(reference "R30")
 					(unit 1)
 				)
@@
 		(dnp no)
 		(fields_autoplaced yes)
-		(property "Reference" "R25"
+		(property "Reference" "R26"
 			(at 80.01 121.9199 0)
 			(show_name no)
@@
 			(project "psu-ext"
 				(path "/3cca1064-5b2a-48a0-8872-f4d00db38e9c/8382cf51-befd-44eb-9cec-01756b7c42d3"
-					(reference "R25")
+					(reference "R26")
 					(unit 1)
 				)
@@
 		(in_pos_files yes)
 		(dnp no)
-		(property "Reference" "R34"
+		(property "Reference" "R35"
 			(at 235.712 38.1 90)
 			(show_name no)
@@
 			(project "psu-ext"
 				(path "/3cca1064-5b2a-48a0-8872-f4d00db38e9c/8382cf51-befd-44eb-9cec-01756b7c42d3"
-					(reference "R34")
+					(reference "R35")
 					(unit 1)
 				)
@@
 		(dnp no)
 		(fields_autoplaced yes)
-		(property "Reference" "R31"
+		(property "Reference" "R32"
 			(at 180.34 53.3399 0)
 			(show_name no)
@@
 			(project "psu-ext"
 				(path "/3cca1064-5b2a-48a0-8872-f4d00db38e9c/8382cf51-befd-44eb-9cec-01756b7c42d3"
-					(reference "R31")
+					(reference "R32")
 					(unit 1)
 				)
@@
 		(in_bom no)
 		(on_board yes)
-		(in_pos_files yes)
+		(in_pos_files no)
 		(dnp no)
 		(property "Reference" "H11"
@@
 		(in_pos_files yes)
 		(dnp no)
-		(property "Reference" "R32"
+		(property "Reference" "R33"
 			(at 189.738 119.888 90)
 			(show_name no)
@@
 			(project "psu-ext"
 				(path "/3cca1064-5b2a-48a0-8872-f4d00db38e9c/8382cf51-befd-44eb-9cec-01756b7c42d3"
-					(reference "R32")
+					(reference "R33")
 					(unit 1)
 				)
@@
 		(dnp no)
 		(fields_autoplaced yes)
-		(property "Reference" "R24"
+		(property "Reference" "R25"
 			(at 45.72 124.46 90)
 			(show_name no)
@@
 			(project "psu-ext"
 				(path "/3cca1064-5b2a-48a0-8872-f4d00db38e9c/8382cf51-befd-44eb-9cec-01756b7c42d3"
-					(reference "R24")
+					(reference "R25")
 					(unit 1)
 				)
@@
 		(in_bom no)
 		(on_board yes)
-		(in_pos_files yes)
+		(in_pos_files no)
 		(dnp no)
 		(property "Reference" "H9"
