File: electronics/psu-ext.kicad_pcb (KiCad board)
At the start: 4 copper layers, 100 x 50 mm, 135 parts, among them J1 TYPE-C-31-M-12, J2 Conn_02x03_Odd_Even, J3 Conn_01x03, K1 HF49FD_005-1H12T, Q1 MMBT2222A, SW1 SW_Push, SW2 SW_Push, U1 USBLC6-2SC6, U10 INA240A2D, U11 TSZ122IYDT, U12 LM2664M6, U2 AP22818AKEWT, U3 LD1117S33, U4 LD1117S33, U5 ESP32-S3-WROOM-1, U6 W25Q16JVSS, U7 ISO1540, U8 ADS1115IDGS, U9 LM321, Y1 FC-135_32.7680KA-A0

Commit message: Added IO3 pullup and negative 3V3 rail testpoint, few other PCB laypu… (#4)
* Added IO3 pullup and negative 3V3 rail testpoint, few other PCB layput improvements.
* Updated exports - gerbers, schematics, bom, CPL KiCad for version 1.3.1

---------

Signed-off-by: Maxim Pavlov <max.eelabs@gmail.com>
Parts:
- removed the R35 at (134.9, 129.7)
- added R14: 10k, Resistor_SMD:R_0805_2012Metric, F.Cu at (193.9, 112.4)
- added R36: 10R, Resistor_SMD:R_0805_2012Metric, B.Cu at (134.9, 129.7)
- added TP7: -3V3, TestPoint:TestPoint_Pad_D1.5mm, F.Cu at (160.0, 112.9)
- C7, C8: value 330p 1kV -> 330p
- D5, D6, D7, D8, D9: value ESD5Zxx -> ESD5Z3.3T1G
- R21: renamed from R20; moved to F.Cu
- R3, R4: value 1k -> 2k
- R31: renamed from R30; value 22k -> 20k
- moved R21 4.41 mm to (182.1, 105.7), turned to 0 degrees
- moved R43 2.00 mm to (157.3, 118.5)
- moved R27 1.31 mm to (165.3, 113.8)
- moved R28 1.31 mm to (163.1, 113.8)
- moved R35 1.14 mm to (156.9, 117.5)
- moved C27 0.68 mm to (158.9, 117.5), turned to 90 degrees
- moved R20 0.25 mm to (190.9, 108.4)
- renumbered R14 to R15, R15 to R16, R16 to R17, R17 to R18, R18 to R19, R19 to R20, R21 to R22, R22 to R23, R23 to R24, R24 to R25, R25 to R26, R26 to R27, R27 to R28, R28 to R29, R29 to R30, R31 to R32, R32 to R33, R33 to R34, R34 to R35, R36 to R37, R37 to R38, R38 to R39, R39 to R40, R40 to R41, R41 to R42, R42 to R43, R43 to R44, R44 to R45, R45 to R46
Connections:
- U5 pad 15: unconnected-(U5-IO3-Pad15) -> Net-(U5-IO3)
Routing:
- net -3V3: track 5.63 -> 14.3 mm, vias 0 -> 1
- net Net-(U6-~{WP}/IO_{2}): track 2.52 -> 8.68 mm, vias 1 -> 2
- net Net-(U5-IO3): track 0.00 -> 3.91 mm
- net Net-(U11A--): track 11.6 -> 10.4 mm
- net /FrontEnd ADC/AIN2: track 8.47 -> 7.63 mm
- net V3.3: track 35.0 -> 35.7 mm, vias 14 -> 15
- net /FrontEnd ADC/SCLS: track 12.0 -> 12.7 mm
