File: electronics/psu-ext.kicad_sch (KiCad schematic)
At the start: 7 parts

Commit message: Added input buffernig and negative rail for near-zero measurments
Added I2C_NUM_1 on IO6 (SDA) and IO7 (SCL).

Signed-off-by: Maxim Pavlov <max.eelabs@gmail.com>
Parts:
- renumbered H5 to H1, H6 to H2, H7 to H3, H8 to H4, H9 to H5, H10 to H6, H11 to H7
Other:
- sheet FrontEnd renamed FrontEnd ADC
- added sheet FrontEnd Volt (front-end-voltage.kicad_sch)
- sheet FrontEnd ADC: file front-end.kicad_sch -> front-end-adc-c.kicad_sch
Changed lines of the file:
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@@
 		(title "PSU-EXT Root")
 		(date "2026-08-08")
-		(rev "1.2.1")
+		(rev "1.3.0")
 		(company "MaxEELabs")
-		(comment 3 "This hardware design is licensed under CERN-OHL-S v2.\nCopyright © 2026 PSU-EXT Authors: https://github.com/PSU-Ext-Org/psu-ext")
+		(comment 3 "This hardware design is licensed under CERN-OHL-S v2.\nCopyright © 2026 PSU-EXT Authors: https://github.com/PSU-Ext-Org")
 	)
 	(text_box "Note: \n\n1uF capactior at EN pint togeter with 10K pullup form RC delay recomended by datasheet\nBoot GIPOS: GPIO0, GPIO3 GPIO45, GPIO046\n\n\nSafe: \nIO4  4  I/O/T RTC_GPIO4,  GPIO4,  TOUCH4, ADC1_CH3\nIO5  5  I/O/T RTC_GPIO5,  GPIO5,  TOUCH5, ADC1_CH4\nIO6  6  I/O/T RTC_GPIO6,  GPIO6,  TOUCH6, ADC1_CH5\nIO7  7  I/O/T RTC_GPIO7,  GPIO7,  TOUCH7, ADC1_CH6\nIO17 10 I/O/T RTC_GPIO17, GPIO17, U1TXD,  ADC2_CH6\n\nExternal Crystal\nIO15 8 I/O/T RTC_GPIO15, GPIO15, U0RTS, ADC2_CH4, XTAL_32K_P\nIO16 9 I/O/T RTC_GPIO16, GPIO16, U0CTS, ADC2_CH5, XTAL_32K_N\n\nMTDI, MTCK, MTMS, and MTDO.\n\nTODO: \n\n- [x] Move Leds to the botton, so there is a place for a crystal\n- [x] Add clock crystal\n- [x] Add voltage measurement - resistor divider to A0\n- [x] Add Jtag port for debug\n- [x] Add protected GPIO \n- [x] Add internal memory\n- [x] Enreach silk-skreen \n- [x] Add testpoints\n- [x] Update JLC BOM\n\n- [x] Test measurement with GND reference (47R + 1nF)\n- [x] Test measuremnt with resistors and cpacitors across 1115\n- [x] Test relay cricuit - if it works\n- [x] Test relay circuit for voltage spikes\n\nTODO Rev 1.1:\n\n- [x] Rename testpoints\n- [x] Add max V and AMP\n- [x] Add led for relay indicator\n- [x] Add OpenHardware logo and MaxEELabs Logo \n- [x] Add Tooling holes\n- [x] Designators Order\n\nTODO Rev 1.2:\n\n- [x] Prepare to CERN-OHL-S v2\n\nNOTE: \nTME 1kV 330pF https://www.tme.eu/pl/en/details/grm31a7u3a331jw31d/mlcc-smd-capacitors/murata/\n"
@@
 		(dnp no)
 		(fields_autoplaced yes)
-		(property "Reference" "H11"
+		(property "Reference" "H7"
 			(at 91.44 92.7099 0)
 			(show_name no)
@@
 			(project "psu-ext"
 				(path "/3cca1064-5b2a-48a0-8872-f4d00db38e9c"
-					(reference "H11")
+					(reference "H7")
 					(unit 1)
 				)
@@
 		(dnp no)
 		(fields_autoplaced yes)
-		(property "Reference" "#PWR05"
+		(property "Reference" "#PWR04"
 			(at 38.1 104.14 0)
 			(hide yes)
@@
 			(project "psu-ext"
 				(path "/3cca1064-5b2a-48a0-8872-f4d00db38e9c"
-					(reference "#PWR05")
+					(reference "#PWR04")
 					(unit 1)
 				)
@@
 		(dnp no)
 		(fields_autoplaced yes)
-		(property "Reference" "#PWR040"
+		(property "Reference" "#PWR02"
 			(at 25.4 104.14 0)
 			(hide yes)
@@
 			(project "psu-ext"
 				(path "/3cca1064-5b2a-48a0-8872-f4d00db38e9c"
-					(reference "#PWR040")
+					(reference "#PWR02")
 					(unit 1)
 				)
@@
 		(dnp no)
 		(fields_autoplaced yes)
-		(property "Reference" "H10"
+		(property "Reference" "H6"
 			(at 66.04 92.7099 0)
 			(show_name no)
@@
 			(project "psu-ext"
 				(path "/3cca1064-5b2a-48a0-8872-f4d00db38e9c"
-					(reference "H10")
+					(reference "H6")
 					(unit 1)
 				)
@@
 		(in_pos_files yes)
 		(dnp no)
-		(property "Reference" "H8"
+		(property "Reference" "H4"
 			(at 38.1 90.17 0)
 			(show_name no)
@@
 			(project "psu-ext"
 				(path "/3cca1064-5b2a-48a0-8872-f4d00db38e9c"
-					(reference "H8")
+					(reference "H4")
 					(unit 1)
 				)
@@
 		(in_pos_files yes)
 		(dnp no)
-		(property "Reference" "H7"
+		(property "Reference" "H3"
 			(at 38.1 72.39 0)
 			(show_name no)
@@
 			(project "psu-ext"
 				(path "/3cca1064-5b2a-48a0-8872-f4d00db38e9c"
-					(reference "H7")
+					(reference "H3")
 					(unit 1)
 				)
@@
 		(dnp no)
 		(fields_autoplaced yes)
-		(property "Reference" "H9"
+		(property "Reference" "H5"
 			(at 66.04 74.9299 0)
 			(show_name no)
@@
 			(project "psu-ext"
 				(path "/3cca1064-5b2a-48a0-8872-f4d00db38e9c"
-					(reference "H9")
+					(reference "H5")
 					(unit 1)
 				)
@@
 		(dnp no)
 		(fields_autoplaced yes)
-		(property "Reference" "#PWR04"
+		(property "Reference" "#PWR03"
 			(at 38.1 86.36 0)
 			(hide yes)
@@
 			(project "psu-ext"
 				(path "/3cca1064-5b2a-48a0-8872-f4d00db38e9c"
-					(reference "#PWR04")
+					(reference "#PWR03")
 					(unit 1)
 				)
@@
 		(dnp no)
 		(fields_autoplaced yes)
-		(property "Reference" "#PWR039"
+		(property "Reference" "#PWR01"
 			(at 25.4 86.36 0)
 			(hide yes)
@@
 			(project "psu-ext"
 				(path "/3cca1064-5b2a-48a0-8872-f4d00db38e9c"
-					(reference "#PWR039")
+					(reference "#PWR01")
 					(unit 1)
 				)
@@
 		(in_pos_files yes)
 		(dnp no)
-		(property "Reference" "H5"
+		(property "Reference" "H1"
 			(at 25.4 72.39 0)
 			(show_name no)
@@
 			(project "psu-ext"
 				(path "/3cca1064-5b2a-48a0-8872-f4d00db38e9c"
-					(reference "H5")
+					(reference "H1")
 					(unit 1)
 				)
@@
 		(in_pos_files yes)
 		(dnp no)
-		(property "Reference" "H6"
+		(property "Reference" "H2"
 			(at 25.4 90.17 0)
 			(show_name no)
@@
 			(project "psu-ext"
 				(path "/3cca1064-5b2a-48a0-8872-f4d00db38e9c"
-					(reference "H6")
+					(reference "H2")
 					(unit 1)
 				)
@@
 	)
 	(sheet
-		(at 25.4 25.4)
+		(at 177.8 25.4)
 		(size 25.4 25.4)
 		(exclude_from_sim no)
@@
 			(color 0 0 0 0)
 		)
-		(property "Sheetname" "USB"
-			(at 25.4 24.6884 0)
+		(property "Sheetname" "FrontEnd Volt"
+			(at 177.8 24.6884 0)
 			(show_name no)
 			(do_not_autoplace no)
@@
 			)
 		)
-		(property "Sheetfile" "usb.kicad_sch"
-			(at 25.4 51.3846 0)
+		(property "Sheetfile" "front-end-voltage.kicad_sch"
+			(at 177.8 51.3846 0)
 			(show_name no)
 			(do_not_autoplace no)
@@
 			(project "psu-ext"
 				(path "/3cca1064-5b2a-48a0-8872-f4d00db38e9c"
-					(page "2")
+					(page "6")
 				)
 			)
@@
 	)
 	(sheet
-		(at 139.7 25.4)
+		(at 25.4 25.4)
 		(size 25.4 25.4)
 		(exclude_from_sim no)
@@
 			(color 0 0 0 0)
 		)
-		(property "Sheetname" "FrontEnd"
+		(property "Sheetname" "USB"
+			(at 25.4 24.6884 0)
+			(show_name no)
+			(do_not_autoplace no)
+			(effects
+				(font
+					(size 1.27 1.27)
+				)
+				(justify left bottom)
+			)
+		)
+		(property "Sheetfile" "usb.kicad_sch"
+			(at 25.4 51.3846 0)
+			(show_name no)
+			(do_not_autoplace no)
+			(effects
+				(font
+					(size 1.27 1.27)
+				)
+				(justify left top)
+			)
+		)
+		(instances
+			(project "psu-ext"
+				(path "/3cca1064-5b2a-48a0-8872-f4d00db38e9c"
+					(page "2")
+				)
+			)
+		)
+	)
+	(sheet
+		(at 139.7 25.4)
+		(size 25.4 25.4)
+		(exclude_from_sim no)
+		(in_bom yes)
+		(on_board yes)
+		(dnp no)
+		(fields_autoplaced yes)
+		(stroke
+			(width 0.1524)
+			(type solid)
+		)
+		(fill
+			(color 0 0 0 0)
+		)
+		(property "Sheetname" "FrontEnd ADC"
 			(at 139.7 24.6884 0)
 			(show_name no)
@@
 			)
 		)
-		(property "Sheetfile" "front-end.kicad_sch"
+		(property "Sheetfile" "front-end-adc-c.kicad_sch"
 			(at 139.7 51.3846 0)
 			(show_name no)
