File: electronics/usb.kicad_sch (KiCad schematic)
At the start: 16 parts, among them J1 TYPE-C-31-M-12, U1 USBLC6-2SC6, U2 AP22818AKEWT

Commit message: Added input buffernig and negative rail for near-zero measurments
Added I2C_NUM_1 on IO6 (SDA) and IO7 (SCL).

Signed-off-by: Maxim Pavlov <max.eelabs@gmail.com>
Parts:
- renumbered R5 to R4, R4 to R5
Changed lines of the file:
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@@
 		(title "PSU-EXT USB")
 		(date "2026-08-08")
-		(rev "1.2.1")
+		(rev "1.3.0")
 		(company "MaxEELabs")
-		(comment 3 "This hardware design is licensed under CERN-OHL-S v2.\nCopyright © 2026 PSU-EXT Authors: https://github.com/PSU-Ext-Org/psu-ext")
+		(comment 3 "This hardware design is licensed under CERN-OHL-S v2.\nCopyright © 2026 PSU-EXT Authors: https://github.com/PSU-Ext-Org")
 	)
 	(junction
@@
 			(justify left bottom)
 		)
-		(property "Net Class" ""
+		(property "Netclass" ""
 			(at 35.56 52.07 0)
 			(show_name no)
@@
 			(justify left bottom)
 		)
-		(property "Net Class" ""
+		(property "Netclass" ""
 			(at 87.63 48.26 0)
 			(show_name no)
@@
 		(in_pos_files yes)
 		(dnp no)
-		(property "Reference" "R5"
+		(property "Reference" "R4"
 			(at 155.956 57.404 90)
 			(show_name no)
@@
 			(project "psu-ext"
 				(path "/3cca1064-5b2a-48a0-8872-f4d00db38e9c/6880c4ba-b120-4f34-82be-c3193c5ae748"
-					(reference "R5")
+					(reference "R4")
 					(unit 1)
 				)
@@
 		(dnp no)
 		(fields_autoplaced yes)
-		(property "Reference" "#PWR025"
+		(property "Reference" "#PWR09"
 			(at 105.41 77.47 0)
 			(hide yes)
@@
 			(project "psu-ext"
 				(path "/3cca1064-5b2a-48a0-8872-f4d00db38e9c/6880c4ba-b120-4f34-82be-c3193c5ae748"
-					(reference "#PWR025")
+					(reference "#PWR09")
 					(unit 1)
 				)
@@
 		(dnp no)
 		(fields_autoplaced yes)
-		(property "Reference" "#PWR027"
+		(property "Reference" "#PWR08"
 			(at 85.09 77.47 0)
 			(hide yes)
@@
 			(project "psu-ext"
 				(path "/3cca1064-5b2a-48a0-8872-f4d00db38e9c/6880c4ba-b120-4f34-82be-c3193c5ae748"
-					(reference "#PWR027")
+					(reference "#PWR08")
 					(unit 1)
 				)
@@
 		(dnp no)
 		(fields_autoplaced yes)
-		(property "Reference" "#PWR023"
+		(property "Reference" "#PWR07"
 			(at 80.01 77.47 0)
 			(hide yes)
@@
 			(project "psu-ext"
 				(path "/3cca1064-5b2a-48a0-8872-f4d00db38e9c/6880c4ba-b120-4f34-82be-c3193c5ae748"
-					(reference "#PWR023")
+					(reference "#PWR07")
 					(unit 1)
 				)
@@
 		(in_pos_files yes)
 		(dnp no)
-		(property "Reference" "R4"
+		(property "Reference" "R5"
 			(at 169.926 42.164 90)
 			(show_name no)
@@
 			(project "psu-ext"
 				(path "/3cca1064-5b2a-48a0-8872-f4d00db38e9c/6880c4ba-b120-4f34-82be-c3193c5ae748"
-					(reference "R4")
+					(reference "R5")
 					(unit 1)
 				)
@@
 		(dnp no)
 		(fields_autoplaced yes)
-		(property "Reference" "#PWR029"
+		(property "Reference" "#PWR05"
 			(at 33.02 30.48 0)
 			(hide yes)
@@
 			(project "psu-ext"
 				(path "/3cca1064-5b2a-48a0-8872-f4d00db38e9c/6880c4ba-b120-4f34-82be-c3193c5ae748"
-					(reference "#PWR029")
+					(reference "#PWR05")
 					(unit 1)
 				)
@@
 		(dnp no)
 		(fields_autoplaced yes)
-		(property "Reference" "#PWR028"
+		(property "Reference" "#PWR06"
 			(at 33.02 77.47 0)
 			(hide yes)
@@
 			(project "psu-ext"
 				(path "/3cca1064-5b2a-48a0-8872-f4d00db38e9c/6880c4ba-b120-4f34-82be-c3193c5ae748"
-					(reference "#PWR028")
+					(reference "#PWR06")
 					(unit 1)
 				)
@@
 		(dnp no)
 		(fields_autoplaced yes)
-		(property "Reference" "#PWR026"
+		(property "Reference" "#PWR011"
 			(at 190.5 77.47 0)
 			(hide yes)
@@
 			(project "psu-ext"
 				(path "/3cca1064-5b2a-48a0-8872-f4d00db38e9c/6880c4ba-b120-4f34-82be-c3193c5ae748"
-					(reference "#PWR026")
+					(reference "#PWR011")
 					(unit 1)
 				)
@@
 		(dnp no)
 		(fields_autoplaced yes)
-		(property "Reference" "#PWR035"
+		(property "Reference" "#PWR010"
 			(at 134.62 77.47 0)
 			(hide yes)
@@
 			(project "psu-ext"
 				(path "/3cca1064-5b2a-48a0-8872-f4d00db38e9c/6880c4ba-b120-4f34-82be-c3193c5ae748"
-					(reference "#PWR035")
+					(reference "#PWR010")
 					(unit 1)
 				)

Commit message: Added IO3 pullup and negative 3V3 rail testpoint, few other PCB layput improvements.
Parts:
- R3: value 1k -> 2.2k
Changed lines of the file:
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@@
 		(title "PSU-EXT USB")
 		(date "2026-08-08")
-		(rev "1.3.0")
+		(rev "1.3.1")
 		(company "MaxEELabs")
 		(comment 3 "This hardware design is licensed under CERN-OHL-S v2.\nCopyright © 2026 PSU-EXT Authors: https://github.com/PSU-Ext-Org")
@@
 			)
 		)
-		(property "Value" "1k"
-			(at 139.446 59.944 90)
-			(show_name no)
-			(do_not_autoplace no)
+		(property "Value" "2.2k"
+			(at 139.446 58.928 90)
+			(show_name no)
+			(do_not_autoplace no)

Commit message: Fixex for proect before PCBA. TODO. BOM, CPL, EXPORT
Parts:
- R3: value 2.2k -> 2k
- R4: value 1k -> 2k
- TP1, TP2, TP3: now left out of the parts list
Changed lines of the file:
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@@
 		(dnp no)
 		(property "Reference" "R4"
-			(at 155.956 57.404 90)
-			(show_name no)
-			(do_not_autoplace no)
-			(effects
-				(font
-					(size 1.27 1.27)
-				)
-			)
-		)
-		(property "Value" "1k"
-			(at 155.956 59.436 90)
+			(at 155.194 57.404 90)
+			(show_name no)
+			(do_not_autoplace no)
+			(effects
+				(font
+					(size 1.27 1.27)
+				)
+			)
+		)
+		(property "Value" "2k"
+			(at 155.194 59.436 90)
 			(show_name no)
 			(do_not_autoplace no)
@@
 			)
 		)
-		(property "Value" "2.2k"
-			(at 139.446 58.928 90)
+		(property "Value" "2k"
+			(at 139.446 59.944 90)
 			(show_name no)
 			(do_not_autoplace no)
@@
 		(body_style 1)
 		(exclude_from_sim no)
-		(in_bom yes)
-		(on_board yes)
-		(in_pos_files yes)
+		(in_bom no)
+		(on_board yes)
+		(in_pos_files no)
 		(dnp no)
 		(property "Reference" "TP1"
@@
 		(body_style 1)
 		(exclude_from_sim no)
-		(in_bom yes)
-		(on_board yes)
-		(in_pos_files yes)
+		(in_bom no)
+		(on_board yes)
+		(in_pos_files no)
 		(dnp no)
 		(fields_autoplaced yes)
@@
 		(body_style 1)
 		(exclude_from_sim no)
-		(in_bom yes)
-		(on_board yes)
-		(in_pos_files yes)
+		(in_bom no)
+		(on_board yes)
+		(in_pos_files no)
 		(dnp no)
 		(fields_autoplaced yes)

Commit message: Replaced USB power switch and refreshed manufacturing exports (#5)
Replaced USB power switch U2 with AP2151DWG-7 (0.8 A). Updated schematic and PCB revision metadata and regenerated the BOM, CPL, schematic PDF, and Gerbers.

Updated CHANGES.txt with the design changes and removed completed export TODOs.

Signed-off-by: Maxim Pavlov <max.eelabs@gmail.com>
Parts:
- U2: value AP22818AKEWT -> AP2151DWG-7
Changed lines of the file:
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@@
 	(title_block
 		(title "PSU-EXT USB")
-		(date "2026-08-08")
-		(rev "1.3.1")
+		(date "2026-10-29")
+		(rev "1.3.2")
 		(company "MaxEELabs")
 		(comment 3 "This hardware design is licensed under CERN-OHL-S v2.\nCopyright © 2026 PSU-EXT Authors: https://github.com/PSU-Ext-Org")
@@
 			)
 		)
-		(property "Value" "AP22818AKEWT"
+		(property "Value" "AP2151DWG-7"
 			(at 190.5 29.21 0)
 			(show_name no)
@@
 			)
 		)
-		(property "Datasheet" "https://www.diodes.com/assets/Datasheets/AP22816_17_18.pdf"
+		(property "Datasheet" "https://www.mouser.pl/datasheet/3/175/1/AP2141D_51D.pdf"
 			(at 190.5 35.56 0)
 			(hide yes)
@@
 			)
 		)
-		(property "Description" "Current limited 2.0A power switch, single channel, SOT-23-5"
+		(property "Description" "Current limited 0.8A power switch, single channel, SOT-23-5"
 			(at 190.5 36.83 0)
 			(hide yes)
